File: GBA SP schematic.brd (EAGLE design)
At the start: 100.5 x 100 mm, 187 parts, among them IC2 FT230XQ, J1 DNP, J11 Debug USB, J12 FPC_14, J13 DNP, J14 FPC_14, J2 MICRO_USB, J4 DNP, J5 DNP, J6 FPC_14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

Commit message: fixing BOM
Parts:
- X, Y: value DNP -> (none)
- moved C47 0.27 mm to (43.1, 90.0), turned to 0 degrees
- moved C49 0.06 mm to (40.3, 90.9), turned to 0 degrees
- moved C14 0.05 mm to (47.9, 90.9), turned to 90 degrees
Connections:
- net 3V3OUT: now also C47.1; no longer C47.2
- net ADAPTER_5V: now also C14.1; no longer C14.2
- net ADAPTER_GND: now also C14.2, C47.2, C49.2; no longer C14.1, C47.1, C49.1
- net MICRO_5V: now also C49.1; no longer C49.2
Routing:
- net ADAPTER_GND: track 15.7 -> 18.0 mm, vias 15 -> 14
